File: Lab4/Lab4 part2.kicad_sch (KiCad schematic)
At the start: 10 parts, among them J1 Conn_01x02_Male, U1 NE555D

Commit message: lab 6.1 update
Parts:
- C1: footprint (none) -> Capacitor_Tantalum_SMD:CP_EIA-3216-18_Kemet-A_Pad1.58x1.35mm_HandSolder
- C2: footprint (none) -> Capacitor_SMD:C_0805_2012Metric_Pad1.18x1.45mm_HandSolder
- D1, D2: footprint (none) -> LED_SMD:LED_1206_3216Metric_Pad1.42x1.75mm_HandSolder
- J1: footprint (none) -> TerminalBlock:TerminalBlock_bornier-2_P5.08mm
- R1, R2, R3, R4: footprint (none) -> Resistor_SMD:R_0805_2012Metric_Pad1.20x1.40mm_HandSolder
Connections:
- net pin_2: now also C1.1, R2.2
- net pin_3: now also R3.2, R4.1
Changed lines of the file:
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@@
+    (effects (font (size 1.27 1.27)) (justify left bottom))
+  )
+  (label "pin_2" (at 60.96 97.79 0)
     (effects (font (size 1.27 1.27)) (justify left bottom))
   )
@@
     (effects (font (size 1.27 1.27)) (justify left bottom))
   )
+  (label "pin_3" (at 180.34 76.2 0)
+    (effects (font (size 1.27 1.27)) (justify left bottom))
+  )
   (label "pin_2" (at 148.59 81.28 0)
     (effects (font (size 1.27 1.27)) (justify left bottom))
@@
   (symbol (lib_id "power:+9V") (at 124.46 25.4 0) (unit 1)
     (in_bom yes) (on_board yes) (fields_autoplaced)
-    (property "Reference" "#PWR?" (id 0) (at 124.46 29.21 0)
+    (property "Reference" "#PWR01" (id 0) (at 124.46 29.21 0)
       (effects (font (size 1.27 1.27)) hide)
     )
     (property "Value" "+9V" (id 1) (at 124.46 20.32 0))
-    (property "Footprint" "" (id 2) (at 124.46 25.4 0)
+    (property "Footprint" "TerminalBlock:TerminalBlock_bornier-2_P5.08mm" (id 2) (at 124.46 25.4 0)
       (effects (font (size 1.27 1.27)) hide)
     )
@@
       (effects (font (size 1.27 1.27)) (justify right))
     )
-    (property "Footprint" "" (id 2) (at 124.46 30.48 0)
+    (property "Footprint" "TerminalBlock:TerminalBlock_bornier-2_P5.08mm" (id 2) (at 124.46 30.48 0)
       (effects (font (size 1.27 1.27)) hide)
     )
@@
       (effects (font (size 1.27 1.27)) (justify right))
     )
-    (property "Footprint" "" (id 2) (at 176.53 107.95 0)
+    (property "Footprint" "LED_SMD:LED_1206_3216Metric_Pad1.42x1.75mm_HandSolder" (id 2) (at 176.53 107.95 0)
       (effects (font (size 1.27 1.27)) hide)
     )
@@
   (symbol (lib_id "power:GND") (at 127 25.4 180) (unit 1)
     (in_bom yes) (on_board yes)
-    (property "Reference" "#PWR?" (id 0) (at 127 19.05 0)
+    (property "Reference" "#PWR02" (id 0) (at 127 19.05 0)
       (effects (font (size 1.27 1.27)) hide)
     )
     (property "Value" "GND" (id 1) (at 129.54 25.4 0))
-    (property "Footprint" "" (id 2) (at 127 25.4 0)
+    (property "Footprint" "TerminalBlock:TerminalBlock_bornier-2_P5.08mm" (id 2) (at 127 25.4 0)
       (effects (font (size 1.27 1.27)) hide)
     )
@@
     (property "Reference" "D1" (id 0) (at 181.61 48.26 90))
     (property "Value" "LED" (id 1) (at 181.61 50.8 90))
-    (property "Footprint" "" (id 2) (at 176.53 48.26 0)
+    (property "Footprint" "LED_SMD:LED_1206_3216Metric_Pad1.42x1.75mm_HandSolder" (id 2) (at 176.53 48.26 0)
       (effects (font (size 1.27 1.27)) hide)
     )
@@
   (symbol (lib_id "power:+9V") (at 69.85 50.8 0) (unit 1)
     (in_bom yes) (on_board yes) (fields_autoplaced)
-    (property "Reference" "#PWR?" (id 0) (at 69.85 54.61 0)
+    (property "Reference" "#PWR04" (id 0) (at 69.85 54.61 0)
       (effects (font (size 1.27 1.27)) hide)
     )
@@
       (effects (font (size 1.27 1.27)) (justify left))
     )
-    (property "Footprint" "" (id 2) (at 174.752 83.82 90)
+    (property "Footprint" "Resistor_SMD:R_0805_2012Metric_Pad1.20x1.40mm_HandSolder" (id 2) (at 174.752 83.82 90)
       (effects (font (size 1.27 1.27)) hide)
     )
@@
       (effects (font (size 1.27 1.27)) (justify left))
     )
-    (property "Footprint" "" (id 2) (at 68.072 54.61 90)
+    (property "Footprint" "Resistor_SMD:R_0805_2012Metric_Pad1.20x1.40mm_HandSolder" (id 2) (at 68.072 54.61 90)
       (effects (font (size 1.27 1.27)) hide)
     )
@@
   (symbol (lib_id "power:+9V") (at 176.53 44.45 0) (unit 1)
     (in_bom yes) (on_board yes) (fields_autoplaced)
-    (property "Reference" "#PWR?" (id 0) (at 176.53 48.26 0)
+    (property "Reference" "#PWR03" (id 0) (at 176.53 48.26 0)
       (effects (font (size 1.27 1.27)) hide)
     )
@@
   (symbol (lib_id "power:GND") (at 121.92 111.76 0) (unit 1)
     (in_bom yes) (on_board yes) (fields_autoplaced)
-    (property "Reference" "#PWR?" (id 0) (at 121.92 118.11 0)
+    (property "Reference" "#PWR06" (id 0) (at 121.92 118.11 0)
       (effects (font (size 1.27 1.27)) hide)
     )
@@
       (effects (font (size 1.27 1.27)) (justify left))
     )
-    (property "Footprint" "" (id 2) (at 70.8152 111.76 0)
+    (property "Footprint" "Capacitor_Tantalum_SMD:CP_EIA-3216-18_Kemet-A_Pad1.58x1.35mm_HandSolder" (id 2) (at 70.8152 111.76 0)
       (effects (font (size 1.27 1.27)) hide)
     )
@@
   (symbol (lib_id "power:+9V") (at 130.81 58.42 0) (unit 1)
     (in_bom yes) (on_board yes) (fields_autoplaced)
-    (property "Reference" "#PWR?" (id 0) (at 130.81 62.23 0)
+    (property "Reference" "#PWR05" (id 0) (at 130.81 62.23 0)
       (effects (font (size 1.27 1.27)) hide)
     )
@@
       (effects (font (size 1.27 1.27)) (justify left))
     )
-    (property "Footprint" "" (id 2) (at 174.752 66.04 90)
+    (property "Footprint" "Resistor_SMD:R_0805_2012Metric_Pad1.20x1.40mm_HandSolder" (id 2) (at 174.752 66.04 90)
       (effects (font (size 1.27 1.27)) hide)
     )
@@
       (effects (font (size 1.27 1.27)) (justify left))
     )
-    (property "Footprint" "" (id 2) (at 89.8652 101.6 0)
+    (property "Footprint" "Capacitor_SMD:C_0805_2012Metric_Pad1.18x1.45mm_HandSolder" (id 2) (at 89.8652 101.6 0)
       (effects (font (size 1.27 1.27)) hide)
     )
@@
       (effects (font (size 1.27 1.27)) (justify left))
     )
-    (property "Footprint" "" (id 2) (at 68.072 83.82 90)
+    (property "Footprint" "Resistor_SMD:R_0805_2012Metric_Pad1.20x1.40mm_HandSolder" (id 2) (at 68.072 83.82 90)
       (effects (font (size 1.27 1.27)) hide)
     )
@@
   (symbol_instances
     (path "/282a963d-bfb8-4d94-9bf6-62b851b06003"
-      (reference "#PWR?") (unit 1) (value "+9V") (footprint "")
+      (reference "#PWR01") (unit 1) (value "+9V") (footprint "TerminalBlock:TerminalBlock_bornier-2_P5.08mm")
     )
     (path "/5d09f4c4-a044-47ca-ac71-306d51ef7f90"
-      (reference "#PWR?") (unit 1) (value "GND") (footprint "")
+      (reference "#PWR02") (unit 1) (value "GND") (footprint "TerminalBlock:TerminalBlock_bornier-2_P5.08mm")
+    )
+    (path "/b412588f-978c-4331-ae0a-8423d483384c"
+      (reference "#PWR03") (unit 1) (value "+9V") (footprint "")
     )
     (path "/74069aab-7706-4166-a931-cdf4c5448779"
-      (reference "#PWR?") (unit 1) (value "+9V") (footprint "")
-    )
-    (path "/b412588f-978c-4331-ae0a-8423d483384c"
-      (reference "#PWR?") (unit 1) (value "+9V") (footprint "")
+      (reference "#PWR04") (unit 1) (value "+9V") (footprint "")
+    )
+    (path "/c17c992d-526c-4279-bbbc-3fdfc491b0ff"
+      (reference "#PWR05") (unit 1) (value "+9V") (footprint "")
     )
     (path "/bcee0015-7b8e-4b42-a656-2b391cf11282"
-      (reference "#PWR?") (unit 1) (value "GND") (footprint "")
-    )
-    (path "/c17c992d-526c-4279-bbbc-3fdfc491b0ff"
-      (reference "#PWR?") (unit 1) (value "+9V") (footprint "")
+      (reference "#PWR06") (unit 1) (value "GND") (footprint "")
     )
     (path "/c045f09e-98f2-4d47-a454-cfd2caa9b0cd"
-      (reference "C1") (unit 1) (value "10uF") (footprint "")
+      (reference "C1") (unit 1) (value "10uF") (footprint "Capacitor_Tantalum_SMD:CP_EIA-3216-18_Kemet-A_Pad1.58x1.35mm_HandSolder")
     )
     (path "/f2108a4f-33f4-402b-a39e-2ed2c2b9e5ee"
-      (reference "C2") (unit 1) (value "0.01uF") (footprint "")
+      (reference "C2") (unit 1) (value "0.01uF") (footprint "Capacitor_SMD:C_0805_2012Metric_Pad1.18x1.45mm_HandSolder")
     )
     (path "/70ae4d7e-4557-4813-8524-16fc63fb4c95"
-      (reference "D1") (unit 1) (value "LED") (footprint "")
+      (reference "D1") (unit 1) (value "LED") (footprint "LED_SMD:LED_1206_3216Metric_Pad1.42x1.75mm_HandSolder")
     )
     (path "/51178cff-09ad-4e7a-93f0-2309be364611"
-      (reference "D2") (unit 1) (value "LED") (footprint "")
+      (reference "D2") (unit 1) (value "LED") (footprint "LED_SMD:LED_1206_3216Metric_Pad1.42x1.75mm_HandSolder")
     )
     (path "/455bb2a7-42c4-4487-b0be-30ab95777f6e"
-      (reference "J1") (unit 1) (value "Conn_01x02_Male") (footprint "")
+      (reference "J1") (unit 1) (value "Conn_01x02_Male") (footprint "TerminalBlock:TerminalBlock_bornier-2_P5.08mm")
     )
     (path "/b3516c82-4832-4970-a96f-5101ef3a446b"
-      (reference "R1") (unit 1) (value "1K") (footprint "")
+      (reference "R1") (unit 1) (value "1K") (footprint "Resistor_SMD:R_0805_2012Metric_Pad1.20x1.40mm_HandSolder")
     )
     (path "/f7a918f5-f477-4015-8f3d-6de4b24bd234"
-      (reference "R2") (unit 1) (value "10K") (footprint "")
+      (reference "R2") (unit 1) (value "10K") (footprint "Resistor_SMD:R_0805_2012Metric_Pad1.20x1.40mm_HandSolder")
     )
     (path "/cf7958ac-92d6-425c-a5fd-922d040e6583"
-      (reference "R3") (unit 1) (value "1K") (footprint "")
+      (reference "R3") (unit 1) (value "1K") (footprint "Resistor_SMD:R_0805_2012Metric_Pad1.20x1.40mm_HandSolder")
     )
     (path "/827a6531-85c1-43f6-8f98-4c6d018c1e71"
-      (reference "R4") (unit 1) (value "1K") (footprint "")
+      (reference "R4") (unit 1) (value "1K") (footprint "Resistor_SMD:R_0805_2012Metric_Pad1.20x1.40mm_HandSolder")
     )
     (path "/bd6c4f52-0425-48a4-8581-a8e7ecb19f1b"
