File: Lab4/Lab4.kicad_sch (KiCad schematic)
At the start: 2 parts

Commit message: lab 6.1 update
Parts:
- added 9V: V1, Connector_JST:JST_PH_B2B-PH-K_1x02_P2.00mm_Vertical, symbol Connector:Conn_01x02_Male
- added C1: 4.7 uF, Capacitor_THT:C_Radial_D5.0mm_H5.0mm_P2.00mm, symbol Device:C_Polarized
- added R2: 2.2 Kohm, Resistor_THT:R_Axial_DIN0516_L15.5mm_D5.0mm_P20.32mm_Horizontal, symbol Device:R
- added SW1: SW_SPDT, Button_Switch_THT:SW_E-Switch_EG1224_SPDT_Angled, symbol Switch:SW_SPDT
- D1: footprint (none) -> LED_THT:LED_D5.0mm
- R1: value 360R -> 20 Kohm; footprint (none) -> Resistor_THT:R_Axial_DIN0516_L15.5mm_D5.0mm_P20.32mm_Horizontal
Connections:
- net GND is gone; now on an unnamed net: R1.2
- net +9V: no longer names the net of D1.2 (A)
- net LED: no longer names the net of D1.1 (K)
- net LED: now also 9V.2 (Pin_2), C1.2; no longer R1.1
- new net: R2.1, SW1.2 (B)
- new net: 9V.1 (Pin_1), R2.2
- new net: C1.1, R1.1, SW1.3 (C)
Changed lines of the file:
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@@
 (kicad_sch (version 20211123) (generator eeschema)
   (paper "A4")
-  (wire (pts (xy 123.19 38.1) (xy 123.19 44.45))
+  (junction (at 135.89 102.87) (diameter 0) (color 0 0 0 0)
+  )
+  (junction (at 135.89 72.39) (diameter 0) (color 0 0 0 0)
+  )
+  (wire (pts (xy 135.89 72.39) (xy 135.89 77.47))
     (stroke (width 0) (type default) (color 0 0 0 0))
   )
-  (wire (pts (xy 91.44 34.29) (xy 91.44 38.1))
+  (wire (pts (xy 166.37 72.39) (xy 135.89 72.39))
     (stroke (width 0) (type default) (color 0 0 0 0))
   )
-  (wire (pts (xy 91.44 45.72) (xy 91.44 48.26))
+  (wire (pts (xy 166.37 99.06) (xy 166.37 102.87))
     (stroke (width 0) (type default) (color 0 0 0 0))
   )
-  (wire (pts (xy 123.19 27.94) (xy 123.19 30.48))
+  (wire (pts (xy 123.19 72.39) (xy 135.89 72.39))
     (stroke (width 0) (type default) (color 0 0 0 0))
   )
-  (label "LED" (at 123.19 27.94 0)
-    (effects (font (size 1.27 1.27)) (justify left bottom))
+  (wire (pts (xy 77.47 69.85) (xy 77.47 95.25))
+    (stroke (width 0) (type default) (color 0 0 0 0))
   )
-  (label "LED" (at 91.44 48.26 0)
-    (effects (font (size 1.27 1.27)) (justify left bottom))
+  (wire (pts (xy 135.89 102.87) (xy 135.89 85.09))
+    (stroke (width 0) (type default) (color 0 0 0 0))
   )
-  (symbol (lib_id "Device:LED") (at 91.44 41.91 90) (unit 1)
+  (wire (pts (xy 166.37 102.87) (xy 135.89 102.87))
+    (stroke (width 0) (type default) (color 0 0 0 0))
+  )
+  (wire (pts (xy 166.37 77.47) (xy 166.37 72.39))
+    (stroke (width 0) (type default) (color 0 0 0 0))
+  )
+  (wire (pts (xy 77.47 102.87) (xy 135.89 102.87))
+    (stroke (width 0) (type default) (color 0 0 0 0))
+  )
+  (wire (pts (xy 166.37 85.09) (xy 166.37 91.44))
+    (stroke (width 0) (type default) (color 0 0 0 0))
+  )
+  (wire (pts (xy 100.33 69.85) (xy 113.03 69.85))
+    (stroke (width 0) (type default) (color 0 0 0 0))
+  )
+  (wire (pts (xy 77.47 97.79) (xy 77.47 102.87))
+    (stroke (width 0) (type default) (color 0 0 0 0))
+  )
+  (wire (pts (xy 77.47 69.85) (xy 92.71 69.85))
+    (stroke (width 0) (type default) (color 0 0 0 0))
+  )
+  (symbol (lib_id "Device:LED") (at 166.37 95.25 90) (unit 1)
     (in_bom yes) (on_board yes) (fields_autoplaced)
-    (property "Reference" "D1" (id 0) (at 95.25 42.2274 90)
+    (property "Reference" "D1" (id 0) (at 170.18 95.5674 90)
       (effects (font (size 1.27 1.27)) (justify right))
     )
-    (property "Value" "LED" (id 1) (at 95.25 44.7674 90)
+    (property "Value" "LED" (id 1) (at 170.18 98.1074 90)
       (effects (font (size 1.27 1.27)) (justify right))
     )
-    (property "Footprint" "" (id 2) (at 91.44 41.91 0)
+    (property "Footprint" "LED_THT:LED_D5.0mm" (id 2) (at 166.37 95.25 0)
       (effects (font (size 1.27 1.27)) hide)
     )
-    (property "Datasheet" "~" (id 3) (at 91.44 41.91 0)
+    (property "Datasheet" "~" (id 3) (at 166.37 95.25 0)
       (effects (font (size 1.27 1.27)) hide)
     )
@@
     (pin "2")
   )
-  (symbol (lib_id "power:GND") (at 123.19 44.45 0) (unit 1)
-    (in_bom yes) (on_board yes) (fields_autoplaced)
-    (property "Reference" "#PWR02" (id 0) (at 123.19 50.8 0)
+  (symbol (lib_id "Device:R") (at 96.52 69.85 270) (unit 1)
+    (in_bom yes) (on_board yes)
+    (property "Reference" "R2" (id 0) (at 95.25 73.66 90)
+      (effects (font (size 1.27 1.27)) (justify left))
+    )
+    (property "Value" "2.2 Kohm" (id 1) (at 92.71 76.2 90)
+      (effects (font (size 1.27 1.27)) (justify left))
+    )
+    (property "Footprint" "Resistor_THT:R_Axial_DIN0516_L15.5mm_D5.0mm_P20.32mm_Horizontal" (id 2) (at 96.52 68.072 90)
       (effects (font (size 1.27 1.27)) hide)
     )
-    (property "Value" "GND" (id 1) (at 123.19 49.53 0))
-    (property "Footprint" "" (id 2) (at 123.19 44.45 0)
-      (effects (font (size 1.27 1.27)) hide)
-    )
-    (property "Datasheet" "" (id 3) (at 123.19 44.45 0)
+    (property "Datasheet" "~" (id 3) (at 96.52 69.85 0)
       (effects (font (size 1.27 1.27)) hide)
     )
     (pin "1")
+    (pin "2")
   )
-  (symbol (lib_id "power:+9V") (at 91.44 34.29 0) (unit 1)
+  (symbol (lib_id "Switch:SW_SPDT") (at 118.11 69.85 0) (unit 1)
     (in_bom yes) (on_board yes) (fields_autoplaced)
-    (property "Reference" "#PWR01" (id 0) (at 91.44 38.1 0)
+    (property "Reference" "SW1" (id 0) (at 118.11 62.23 0))
+    (property "Value" "SW_SPDT" (id 1) (at 118.11 64.77 0))
+    (property "Footprint" "Button_Switch_THT:SW_E-Switch_EG1224_SPDT_Angled" (id 2) (at 118.11 69.85 0)
       (effects (font (size 1.27 1.27)) hide)
     )
-    (property "Value" "+9V" (id 1) (at 91.44 29.21 0))
-    (property "Footprint" "" (id 2) (at 91.44 34.29 0)
-      (effects (font (size 1.27 1.27)) hide)
-    )
-    (property "Datasheet" "" (id 3) (at 91.44 34.29 0)
+    (property "Datasheet" "~" (id 3) (at 118.11 69.85 0)
       (effects (font (size 1.27 1.27)) hide)
     )
     (pin "1")
+    (pin "2")
+    (pin "3")
   )
-  (symbol (lib_id "Device:R") (at 123.19 34.29 0) (unit 1)
+  (symbol (lib_id "Device:C_Polarized") (at 135.89 81.28 0) (unit 1)
     (in_bom yes) (on_board yes) (fields_autoplaced)
-    (property "Reference" "R1" (id 0) (at 125.73 33.0199 0)
+    (property "Reference" "C1" (id 0) (at 139.7 79.1209 0)
       (effects (font (size 1.27 1.27)) (justify left))
     )
-    (property "Value" "360R" (id 1) (at 125.73 35.5599 0)
+    (property "Value" "4.7 uF" (id 1) (at 139.7 81.6609 0)
       (effects (font (size 1.27 1.27)) (justify left))
     )
-    (property "Footprint" "" (id 2) (at 121.412 34.29 90)
+    (property "Footprint" "Capacitor_THT:C_Radial_D5.0mm_H5.0mm_P2.00mm" (id 2) (at 136.8552 85.09 0)
       (effects (font (size 1.27 1.27)) hide)
     )
-    (property "Datasheet" "~" (id 3) (at 123.19 34.29 0)
+    (property "Datasheet" "~" (id 3) (at 135.89 81.28 0)
+      (effects (font (size 1.27 1.27)) hide)
+    )
+    (pin "1")
+    (pin "2")
+  )
+  (symbol (lib_id "Device:R") (at 166.37 81.28 0) (unit 1)
+    (in_bom yes) (on_board yes) (fields_autoplaced)
+    (property "Reference" "R1" (id 0) (at 168.91 80.0099 0)
+      (effects (font (size 1.27 1.27)) (justify left))
+    )
+    (property "Value" "20 Kohm" (id 1) (at 168.91 82.5499 0)
+      (effects (font (size 1.27 1.27)) (justify left))
+    )
+    (property "Footprint" "Resistor_THT:R_Axial_DIN0516_L15.5mm_D5.0mm_P20.32mm_Horizontal" (id 2) (at 164.592 81.28 90)
+      (effects (font (size 1.27 1.27)) hide)
+    )
+    (property "Datasheet" "~" (id 3) (at 166.37 81.28 0)
+      (effects (font (size 1.27 1.27)) hide)
+    )
+    (pin "1")
+    (pin "2")
+  )
+  (symbol (lib_id "Connector:Conn_01x02_Male") (at 72.39 95.25 0) (unit 1)
+    (in_bom yes) (on_board yes) (fields_autoplaced)
+    (property "Reference" "9V" (id 0) (at 73.025 90.17 0))
+    (property "Value" "V1" (id 1) (at 73.025 92.71 0))
+    (property "Footprint" "Connector_JST:JST_PH_B2B-PH-K_1x02_P2.00mm_Vertical" (id 2) (at 72.39 95.25 0)
+      (effects (font (size 1.27 1.27)) hide)
+    )
+    (property "Datasheet" "~" (id 3) (at 72.39 95.25 0)
       (effects (font (size 1.27 1.27)) hide)
     )
@@
   )
   (symbol_instances
-    (path "/69fcd4af-ea9c-44ca-be18-f9f45b6073b5"
-      (reference "#PWR01") (unit 1) (value "+9V") (footprint "")
+    (path "/7af85083-f579-4058-aa6c-ba496da592ba"
+      (reference "9V") (unit 1) (value "V1") (footprint "Connector_JST:JST_PH_B2B-PH-K_1x02_P2.00mm_Vertical")
     )
-    (path "/147c724b-6831-4bf5-9aee-1752544ab419"
-      (reference "#PWR02") (unit 1) (value "GND") (footprint "")
+    (path "/4e653426-895c-43ec-96ae-d39c1b4fc6d5"
+      (reference "C1") (unit 1) (value "4.7 uF") (footprint "Capacitor_THT:C_Radial_D5.0mm_H5.0mm_P2.00mm")
     )
-    (path "/0b408de4-68b0-4f86-90da-8f0cc8e34e5d"
-      (reference "D1") (unit 1) (value "LED") (footprint "")
+    (path "/1f10b459-2e5a-4681-b246-ce4be7f7d93b"
+      (reference "D1") (unit 1) (value "LED") (footprint "LED_THT:LED_D5.0mm")
     )
-    (path "/b6dc29eb-c8ca-4eb6-af57-ea43d53cb0a4"
-      (reference "R1") (unit 1) (value "360R") (footprint "")
+    (path "/5e223131-6999-40c1-bba7-50b7da2315c1"
+      (reference "R1") (unit 1) (value "20 Kohm") (footprint "Resistor_THT:R_Axial_DIN0516_L15.5mm_D5.0mm_P20.32mm_Horizontal")
+    )
+    (path "/2b8e4e6f-e7cb-4dbc-94db-6fdfbf1a7a61"
+      (reference "R2") (unit 1) (value "2.2 Kohm") (footprint "Resistor_THT:R_Axial_DIN0516_L15.5mm_D5.0mm_P20.32mm_Horizontal")
+    )
+    (path "/3a7e590a-f09c-4b3d-b6d3-1f6cc004e47a"
+      (reference "SW1") (unit 1) (value "SW_SPDT") (footprint "Button_Switch_THT:SW_E-Switch_EG1224_SPDT_Angled")
     )
   )

Commit message: update lab6 part 2
Parts:
- renumbered 9V to 9V1
Changed lines of the file:
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@@
   (symbol (lib_id "Connector:Conn_01x02_Male") (at 72.39 95.25 0) (unit 1)
     (in_bom yes) (on_board yes) (fields_autoplaced)
-    (property "Reference" "9V" (id 0) (at 73.025 90.17 0))
+    (property "Reference" "9V1" (id 0) (at 73.025 90.17 0))
     (property "Value" "V1" (id 1) (at 73.025 92.71 0))
     (property "Footprint" "Connector_JST:JST_PH_B2B-PH-K_1x02_P2.00mm_Vertical" (id 2) (at 72.39 95.25 0)
@@
   (symbol_instances
     (path "/7af85083-f579-4058-aa6c-ba496da592ba"
-      (reference "9V") (unit 1) (value "V1") (footprint "Connector_JST:JST_PH_B2B-PH-K_1x02_P2.00mm_Vertical")
+      (reference "9V1") (unit 1) (value "V1") (footprint "Connector_JST:JST_PH_B2B-PH-K_1x02_P2.00mm_Vertical")
     )
     (path "/4e653426-895c-43ec-96ae-d39c1b4fc6d5"
